File: FishIoT/FishIoT.kicad_sch (KiCad schematic)
At the start: 123 parts, among them IC1 RV-3032-C7_32.768KHZ-2.5PPM-T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, J1 VDD_JUMPER, J10 RM_UART, J2 0705430001, J3 SF72S006VBDR2500, J4 SHF-105-01-L-D-SM, J5 10119313-302TLF, J6 Conn_01x02_Socket, J7 Conn_01x02_Socket, J8 BM05B-ZESS-TBT, J9 SHF-105-01-L-D-SM, SW1 PTS645SM43SMTR92 LF, SW2 PTS645SM43SMTR92 LF, SW3 PTS645SM43SMTR92 LF, U1 NRF9160-SICA, U10 RM126x, U2 SKY65943-11, U3 TPD3F303DPVR, U4 TPS63000, U5 USBLC6-2P6, U6 CP2102N-Axx-xQFN20, U7 NX3020NAKV, U8 NX3020NAKV, U9 MAX3471

Commit message: Changed GNSS antenna into u.fl. connector, decreased size of pcb further
Parts:
- removed C32: PHVL-3R9V255-R, FishIoT_Footprint_library:PHVL3R9V255R, symbol Device:C_Polarized
- removed E1: DSGP.1575.18.4.A.02, FishIoT_Footprint_library:XCVR_DSGP.1575.18.4.A.02, symbol FishIoTSymbol_Library.Library:DSGP.1575.18.4.A.02
- removed J6, J7: Conn_01x02_Socket, Connector_PinHeader_2.54mm:PinHeader_1x02_P2.54mm_Vertical, symbol Connector:Conn_01x02_Socket
- removed J9: SHF-105-01-L-D-SM, FishIoT_Footprint_library:SHF-105-01-X-D-SM, symbol FishIoTSymbol_Library.Library:SHF-105-01-L-D-SM
- removed R16, R17, R18, R19: 1M, Resistor_SMD:R_0603_1608Metric, symbol Device:R
- added C32: 0.1u, Capacitor_SMD:C_0603_1608Metric, symbol Device:C
- added H1, H2: MountingHole_Pad, MountingHole:MountingHole_3mm_Pad_Via, symbol Mechanical:MountingHole_Pad
- added J11: Current Measurement, Connector_PinHeader_2.54mm:PinHeader_1x02_P2.54mm_Horizontal, symbol Connector:Conn_01x02_Pin
- added J13: UART_DEBUG, Connector_PinHeader_2.54mm:PinHeader_1x03_P2.54mm_Vertical, symbol Connector:Conn_01x03_Socket
- added J9: Conn_Coaxial, FishIoT_Footprint_library:LINX_CONUFL001-SMD-T, symbol Connector:Conn_Coaxial
- R27: footprint Resistor_SMD:R_0201_0603Metric -> Resistor_SMD:R_0603_1608Metric
- R34, R35: value 680 -> 10k
Connections:
- net +3V3: now also R34.2, C32.2
- net GND: now also R35.1, C32.1, J13.1 (Pin_1), J9.2 (Ext)
- net GPS_RF_ANT: now also J9.1 (In)
- net VREG_IN: now also J11.2 (Pin_2); no longer J1.2 (Pin_2)
- net nRF_UART_RX: now also J13.2 (Pin_2)
- net nRF_UART_TX: now also J13.3 (Pin_3)
- net RM_SWCLK: no longer names the net of U10.37 (PA01)
- net RM_SWDIO: no longer names the net of U10.38 (PA02)
- net RM_SWO: no longer names the net of U10.39 (PA03)
- new net VIN: J1.2 (Pin_2), J11.1 (Pin_1)
Other:
- note added: "MountingHoles"
- note added: "Should use jumper"
- moved on the sheet: J1, J10, R34, R35

Commit message: updated schematic and pcb
Parts:
- removed C3: N.C., Capacitor_SMD:C_0603_1608Metric, symbol Device:C
- removed C4: 3.5pF, Capacitor_SMD:C_0603_1608Metric, symbol Device:C
- removed R28: 10k, Resistor_SMD:R_0603_1608Metric, symbol Device:R
- added BT1: 3002, FishIoT_Footprint_library:BAT_3002, symbol FishIoTSymbol_Library.Library:3002
- added H3: MountingHole_Pad, MountingHole:MountingHole_3mm_Pad_Via, symbol Mechanical:MountingHole_Pad
- added L3: L, Inductor_SMD:L_0603_1608Metric, symbol Device:L
- added L4: 33nH, Inductor_SMD:L_0603_1608Metric, symbol Device:L
- added R16: R, Resistor_SMD:R_0603_1608Metric, symbol Device:R
- added R17: 120, Resistor_SMD:R_0603_1608Metric, symbol Device:R
- C1: value N.C. -> C
- C2: value N.C. -> 100n
- C33: value 100n -> 0.1u
- R5: value 180 -> 120
- RTC_EVI1: renamed from TP11; value TestPoint -> RTC_EVI
- renumbered TP6 to PPS1, TP13 to RS_A1, TP14 to RS_B1, TP12 to RTC_CO1, TP10 to SCL1, TP9 to SDA1, TP3 to SWDCLK1, TP2 to SWDIO1, TP15 to TBR_PPS1, TP4 to VSIM1, TP8 to Vbat1, TP5 to Vgpio1, TP1 to Vin1, TP7 to Vout1
Connections:
- net +3V3: now also L4.2
- net GND: now also C2.1, H1.1, H2.1, BT1.N, H3.1, L3.1; no longer C2.2
- net GPS_RF_ANT: now also L3.2, R16.1; no longer J9.1 (In)
- net LTE_RF1: no longer C1.1
- net at L1.2: now also ANT1.1 (FEED), L2.2; no longer C2.1
- net at IC1.1 (VBACKUP): now also C2.2, R17.2
- new net: C1.1, J9.1 (In), L4.1, R16.2
- new net: BT1.P1, R17.1
Other:
- moved on the sheet: IC1, R31, R32, R33, RTC_CO1, RTC_EVI1

Commit message: removed MOS for leds, added RS connector
Parts:
- removed TBR_PPS1: TestPoint, TestPoint:TestPoint_Pad_D1.0mm, symbol Connector:TestPoint
- removed U7, U8: NX3020NAKV, Package_TO_SOT_SMD:SOT-666, symbol FishIoTSymbol_Library.Library:NX3020NAKV
- added J6: BM05B-ZESS-TBT, FishIoT_Footprint_library:BM05BZESSTBTLFSN, symbol Connector:Conn_01x05_Socket
- J11: footprint Connector_PinHeader_2.54mm:PinHeader_1x02_P2.54mm_Horizontal -> Connector_PinHeader_2.54mm:PinHeader_1x02_P2.54mm_Vertical
- renumbered D4 to D1, D5 to D2, D2 to D3, D3 to D4, D1 to D5, R22 to R20, R23 to R21, R20 to R22, R21 to R23
Connections:
- net nRF91_LED1: now also D1.1 (K)
- net nRF91_LED2: now also D2.1 (K)
- net nRF91_LED3: now also D3.1 (K)
- net nRF91_LED4: now also D4.1 (K)
Other:
- moved on the sheet: D1, D2, R20, R21

Commit message: Fixed a bug on batteryvoltage for ADC input pin
Parts:
- added L7: 33nH, Inductor_SMD:L_0603_1608Metric, symbol Device:L
Connections:
- net Battery_voltage: now also U1.23 (P0.13/AIN0); no longer U1.19 (P0.11)
- net GND: now also J6.4 (Pin_4)
- net GPS_EN: now also L7.1
- net VREG_IN: now also J6.1 (Pin_1)
- net at C1.1, J9.1 (In), L4.1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: now also L7.2
- net UART1_TX: now reaches J6.2 (Pin_2)
- net UART1_TX: now also U1.15 (P0.08)
- net UART1_RX: now reaches J6.3 (Pin_3)
- net UART1_RX: now also U1.16 (P0.09)
Other:
- note added: "Auxillary UART"
- moved on the sheet: H1, H2, H3, J6, J8, L4
